File: pwm_driver_kicad/pwm_driver_kicad.kicad_pcb (KiCad board)
At the start: 2 copper layers, 35 x 35 mm, 10 parts, among them J1 Bornera, Q1 IRF1407, U1 NE555P

Commit message: Set correct 3d models path
Routing:
- added copper zone on B.Cu, net 0
Other:
- board text added: "PWM Driver"
- board text removed: "Driver PWM"
Changed lines of the file:
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@@
   (setup
     (pad_to_mask_clearance 0)
+    (grid_origin 104.9865 80)
     (pcbplotparams
       (layerselection 0x00010fc_ffffffff)
@@
     (pad "3" thru_hole oval (at 10 0 90) (size 1.98 3.96) (drill 1.32) (layers "*.Cu" "*.Mask")
       (net 5 "VCC") (pinfunction "Pin_1") (pintype "passive"))
-    (model "${KICAD6_3DMODEL_DIR}/TerminalBlock.3dshapes/TerminalBlock_Altech_AK300-3_P5.00mm.wrl"
-      (offset (xyz 0 0 0))
-      (scale (xyz 1 1 1))
-      (rotate (xyz 0 0 0))
-    )
-    (model "/home/mk/dox/fiuba/86.70/driver_led_integrador/screw-terminal-dg-301-5mm-1.snapshot.1/dg-301-5_0.step"
+    (model "/home/mk/dox/fiuba/86.70/driver_led_integrador/3d_models/screw-terminal-dg-301-5mm-1.snapshot.1/dg-301-5_0.step"
       (offset (xyz -2.5 -3 0))
       (scale (xyz 1 1 1))
@@
     (pad "3" thru_hole circle (at 0 10 180) (size 3 3) (drill 1.2) (layers "*.Cu" "*.Mask")
       (net 3 "Net-(D1-K)") (pinfunction "3") (pintype "passive"))
-    (model "${KICAD6_3DMODEL_DIR}/Potentiometer_THT.3dshapes/Potentiometer_Alps_RK163_Single_Horizontal.wrl"
-      (offset (xyz 0 0 0))
-      (scale (xyz 1 1 1))
-      (rotate (xyz 0 0 0))
-    )
-    (model "/home/mk/dox/fiuba/86.70/driver_led_integrador/alpha-rv16af-20-1.snapshot.9/RV16AF-20.step"
+    (model "/home/mk/dox/fiuba/86.70/driver_led_integrador/3d_models/alpha-rv16af-20-1.snapshot.9/RV16AF-20.step"
       (offset (xyz 7 -5 12.5))
       (scale (xyz 1 1 1))
@@
     (effects (font (size 1.25 1.25) (thickness 0.15)) (justify right bottom))
   )
-  (gr_text "Driver\nPWM" (at 115.8 45.55 180) (layer "F.SilkS")
+  (gr_text "PWM\nDriver" (at 114.75 46.1 180) (layer "F.SilkS")
     (effects (font (size 1.5 1.5) (thickness 0.15)) (justify bottom))
   )
@@
     (effects (font (size 1.5 1.5) (thickness 0.3) bold) (justify left bottom))
   )
-  (gr_text "kloeckner.com.ar" (at 110.9 78.8) (layer "F.SilkS")
+  (gr_text "kloeckner.com.ar" (at 111.5365 78.75) (layer "F.SilkS")
     (effects (font (size 1.75 1.75) (thickness 0.15)) (justify left bottom))
   )
@@
   (segment (start 124.9865 71) (end 125.5865 71.6) (width 0.508) (layer "B.Cu") (net 10))
   (segment (start 130.0865 71.6) (end 136.1865 65.5) (width 0.508) (layer "B.Cu") (net 10))
+  (zone (net 2) (net_name "0") (layer "B.Cu") (hatch edge 0.5)
+    (connect_pads (clearance 0.5))
+    (min_thickness 0.25) (filled_areas_thickness no)
+    (fill yes (thermal_gap 0.5) (thermal_bridge_width 0.5) (island_removal_mode 1) (island_area_min 10))
+    (polygon
+      (pts
+        (xy 104.95 45)
+        (xy 104.95 77.7)
+        (xy 107.3 80.05)
+        (xy 138 80.05)
+        (xy 140 78.05)
+        (xy 140 47.35)
+        (xy 137.65 45)
+        (xy 107.05 45)
+        (xy 105 47.05)
+        (xy 105 45.05)
+      )
+    )
+  )
 )
