File: pwm_driver_kicad/pwm_driver_kicad.kicad_pcb (KiCad board)
At the start: 2 copper layers, 35 x 35 mm, 10 parts, among them J1 Bornera, Q1 IRF1407, U1 NE555P

Commit message: update schematic resistor values | fix simulation
NOTE: the pcb has **not** been updated yet
Parts:
- Q1: footprint Package_TO_SOT_THT:TO-220-3_Vertical -> Library:TO-220-3_Vertical_G_D_S_order
- moved C1 1.55 mm to (128.5, 58.5)
- moved R1 1.29 mm to (118.1, 69.1)
- moved R2 1.23 mm to (130.2, 47.8)
- moved Q1 1.21 mm to (124.9, 72.7)
- moved D2 1.10 mm to (126.2, 51.1)
- moved D1 0.60 mm to (118.5, 54.1)
- moved U1 0.19 mm to (117.9, 64.7)
Routing:
- net Net-(U1-THR): track 39.6 -> 0.00 mm
- net Net-(D1-K): track 16.8 -> 0.00 mm
- net Net-(D1-A): track 13.0 -> 0.55 mm
- net Net-(D2-A): track 11.3 -> 0.00 mm
- net VCC: track 47.8 -> 38.6 mm
- net Net-(J1-Pin_3): track 14.0 -> 21.3 mm
- net Net-(Q1-G): track 6.00 -> 0.00 mm
- net Net-(U1-Q): track 5.71 -> 0.12 mm
- net Net-(U1-CV): track 4.01 -> 0.16 mm
- net 0: track 35.3 -> 38.9 mm
- removed copper zone on B.Cu, net 0
Other:
- board text added: "M. J. Klöckner"
- board text removed: "kloeckner.com.ar"

Commit message: update pcb from schematic
Parts:
- Q1: footprint Library:TO-220-3_Vertical_G_D_S_order -> Package_TO_SOT_THT:TO-220-3_Vertical
- R1: value 46k -> 10k
- moved R1 16.0 mm to (131.8, 77.5), turned to 180 degrees
- moved Q1 5.72 mm to (130.5, 71.5)
- moved D2 4.56 mm to (122.8, 48.0)
- moved D1 4.20 mm to (115.2, 51.5)
- moved R2 3.37 mm to (133.6, 48.0)
- moved U1 1.30 mm to (117.7, 66.0)
- moved C2 1.25 mm to (110.0, 73.0)
Connections:
- C1 pad 2: 0 -> GND
- C2 pad 2: 0 -> GND
- J1 pad 2: 0 -> GND
- Q1 pad 3: 0 -> GND
- R1 pad 1: Net-(U1-Q) -> Net-(Q1-G)
- R1 pad 2: Net-(Q1-G) -> GND
- U1 pad 1: 0 -> GND
- U1 pad 3: Net-(U1-Q) -> Net-(Q1-G)
Routing:
- net GND: track 0.00 -> 45.5 mm
- net Net-(U1-THR): track 0.00 -> 40.6 mm
- net 0: track 38.9 -> 0.00 mm
- net Net-(D1-A): track 0.55 -> 28.1 mm
- net Net-(Q1-G): track 0.00 -> 21.8 mm
- net Net-(D1-K): track 0.00 -> 18.0 mm
- net Net-(J1-Pin_3): track 21.3 -> 8.36 mm
- net Net-(D2-A): track 0.00 -> 11.4 mm
- net VCC: track 38.6 -> 43.9 mm
- net Net-(U1-CV): track 0.16 -> 3.23 mm
- added copper zone on B.Cu, net GND
Other:
- board text added: "Klöckner"
- board text removed: "M. J. Klöckner"

Commit message: fix mosfet footprint pinout
Parts:
- Q1: value IRF1407 -> IRF540
- moved R1 9.60 mm to (125.8, 70.0)
- moved Q1 6.79 mm to (125.4, 76.0), turned to 0 degrees
- moved R2 1.62 mm to (133.0, 49.5)
- moved D1 1.12 mm to (114.2, 51.0)
- moved D2 1.12 mm to (121.8, 47.5)
Routing:
- net GND: track 45.5 -> 23.2 mm
- net Net-(Q1-G): track 21.8 -> 11.9 mm
- net Net-(J1-Pin_3): track 8.36 -> 13.9 mm
- net VCC: track 43.9 -> 42.6 mm
- net Net-(D1-A): track 28.1 -> 29.1 mm
- removed copper zone on B.Cu, net GND

Commit message: update pcb layout
Routing:
- added copper zone on B.Cu, net GND
Changed lines of the file:
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@@
 		(net 9)
 	)
+	(zone
+		(net 8)
+		(net_name "GND")
+		(layer "B.Cu")
+		(hatch edge 0.5)
+		(connect_pads
+			(clearance 0.5)
+		)
+		(min_thickness 0.25)
+		(filled_areas_thickness no)
+		(fill yes
+			(thermal_gap 0.5)
+			(thermal_bridge_width 0.5)
+		)
+		(polygon
+			(pts
+				(xy 104.9865 45) (xy 139.9865 45) (xy 139.9865 80) (xy 104.9865 80)
+			)
+		)
+	)
 )

Commit message: replace third party 3D potentiometer model with own design
Parts:
- moved Q1 0.50 mm to (125.4, 76.5)
Other:
- board text added: "- +"
- board text added: "PWM-"
- board text removed: "-PWM - +"
- board text removed: "max 18V"
Changed lines of the file:
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@@
 		)
 		(fp_text user "K"
-			(at -1.685 1.5 0)
+			(at -1.935 0 0)
 			(layer "F.SilkS")
 			(effects
@@
 	(footprint "Package_TO_SOT_THT:TO-220-3_Vertical"
 		(layer "F.Cu")
-		(at 125.4065 76)
+		(at 125.4065 76.5)
 		(descr "TO-220-3, Vertical, RM 2.54mm, see https://www.vishay.com/docs/66542/to-220-1.pdf")
 		(tags "TO-220-3 Vertical RM 2.54mm")
 		(property "Reference" "Q1"
-			(at 2.54 -4.27 0)
+			(at 2.54 -5 0)
 			(layer "F.SilkS")
 			(effects
@@
 		)
 		(fp_text user "K"
-			(at -1.8715 -0.05 0)
+			(at -2.185 0 0)
 			(layer "F.SilkS")
 			(effects
@@
 		)
 		(model "${KIPRJMOD}/pwm_driver_3d_models/alpha-rv16af-20-1.snapshot.9/RV16AF-20.step"
+			(hide yes)
 			(offset
 				(xyz 7 -5 12.5)
@@
 			)
 		)
+		(model "${KIPRJMOD}/pwm_driver_3d_models/potentiometer_propio.step"
+			(offset
+				(xyz -0.5 -5 14)
+			)
+			(scale
+				(xyz 1 1 1)
+			)
+			(rotate
+				(xyz -90 0 90)
+			)
+		)
 	)
 	(footprint "Package_DIP:DIP-8_W7.62mm"
@@
 		(layer "Edge.Cuts")
 	)
-	(gr_text "max\n18V"
-		(at 138.7 69.4 90)
+	(gr_text "PWM-"
+		(at 132.9865 67.75 90)
 		(layer "F.SilkS")
 		(effects
 			(font
-				(size 1.25 1.25)
+				(size 1 1)
 				(thickness 0.15)
 			)
-			(justify right bottom)
+			(justify left bottom)
 		)
 	)
 	(gr_text "PWM Driver"
-		(at 122.4865 54 180)
+		(at 122.9865 53.5 180)
 		(layer "F.SilkS")
 		(effects
@@
 		)
 	)
-	(gr_text "-PWM  -   +"
-		(at 132 70.9 90)
+	(gr_text "       -   +"
+		(at 133.2365 69.75 90)
 		(layer "F.SilkS")
 		(effects
@@
 	)
 	(gr_text "Klöckner"
-		(at 110.4865 77.5 0)
+		(at 110.7365 78.25 0)
 		(layer "F.SilkS")
 		(effects
 			(font
-				(size 1.75 1.75)
+				(size 1.5 1.5)
 				(thickness 0.15)
 			)
