File: pwm_driver_kicad/pwm_driver_kicad.kicad_sch (KiCad schematic)
At the start: 11 parts, among them J1 Bornera, Q1 IRF1407, U1 NE555P

Commit message: update schematic resistor values | fix simulation
NOTE: the pcb has **not** been updated yet
Parts:
- removed R1: 46k, Resistor_THT:R_Axial_DIN0207_L6.3mm_D2.5mm_P7.62mm_Horizontal, symbol Device:R_US
Connections:
- net 0: no longer C1.2, C2.2, J1.2 (Pin_2), Q1.3 (S), U1.1 (GND)
- net at U1.3 (Q): now also Q1.2 (G)
- new net GND: C1.2, C2.2, J1.2 (Pin_2), Q1.3 (S), U1.1 (GND)
Other:
- moved on the sheet: B1, C1, C2, D1, D2, J1, Q1, R2, RV1, U1

Commit message: add transistor gate pulldown resistor
Parts:
- added R1: 10k, Resistor_THT:R_Axial_DIN0207_L6.3mm_D2.5mm_P7.62mm_Horizontal, symbol Device:R_US
Connections:
- net 0 is gone; now on net GND: B1.2 (N-)
- net GND: now also R1.2
- net at Q1.2 (G), U1.3 (Q): now also R1.1
Other:
- moved on the sheet: Q1
Changed lines of the file:
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@@
+	)
+	(junction
+		(at 171.45 95.25)
+		(diameter 0)
+		(color 0 0 0 0)
+	)
+	(junction
+		(at 171.45 102.87)
+		(diameter 0)
+		(color 0 0 0 1)
+	)
+	(junction
+		(at 168.91 102.87)
+		(diameter 0)
+		(color 0 0 0 1)
 	)
 	(junction
@@
 		(at 160.02 119.38)
 		(diameter 0)
-		(color 0 0 0 0)
+		(color 0 0 0 1)
 	)
 	(junction
 		(at 133.35 119.38)
 		(diameter 0)
-		(color 0 0 0 0)
-	)
-	(junction
-		(at 168.91 104.14)
-		(diameter 0)
-		(color 0 0 0 0)
+		(color 0 0 0 1)
 	)
 	(junction
@@
 	(wire
 		(pts
+			(xy 171.45 102.87) (xy 181.61 102.87)
+		)
+		(stroke
+			(width 0)
+			(type default)
+			(color 0 0 0 1)
+		)
+	)
+	(wire
+		(pts
 			(xy 160.02 85.09) (xy 160.02 86.36)
 		)
@@
 	(wire
 		(pts
-			(xy 177.8 87.63) (xy 171.45 87.63)
-		)
-		(stroke
-			(width 0)
-			(type default)
-		)
-	)
-	(wire
-		(pts
-			(xy 177.8 87.63) (xy 177.8 90.17)
+			(xy 181.61 87.63) (xy 171.45 87.63)
+		)
+		(stroke
+			(width 0)
+			(type default)
+		)
+	)
+	(wire
+		(pts
+			(xy 181.61 87.63) (xy 181.61 90.17)
 		)
 		(stroke
@@
 	(wire
 		(pts
-			(xy 177.8 100.33) (xy 177.8 104.14)
+			(xy 181.61 100.33) (xy 181.61 102.87)
 		)
 		(stroke
@@
 	(wire
 		(pts
-			(xy 146.05 95.25) (xy 170.18 95.25)
+			(xy 146.05 95.25) (xy 171.45 95.25)
 		)
 		(stroke
@@
 	(wire
 		(pts
-			(xy 168.91 104.14) (xy 168.91 119.38)
+			(xy 168.91 102.87) (xy 168.91 119.38)
 		)
 		(stroke
@@
 			(width 0)
 			(type default)
+			(color 255 0 0 1)
+		)
+	)
+	(wire
+		(pts
+			(xy 171.45 95.25) (xy 173.99 95.25)
+		)
+		(stroke
+			(width 0)
+			(type default)
 		)
 	)
@@
 	(wire
 		(pts
-			(xy 168.91 104.14) (xy 177.8 104.14)
+			(xy 168.91 102.87) (xy 171.45 102.87)
 		)
 		(stroke
@@
 	(wire
 		(pts
-			(xy 168.91 83.82) (xy 168.91 104.14)
+			(xy 168.91 83.82) (xy 168.91 102.87)
 		)
 		(stroke
@@
 		(exclude_from_sim no)
 		(in_bom yes)
-		(on_board yes)
+		(on_board no)
 		(dnp no)
 		(property "Reference" "B1"
@@
 				(path "/d8411f75-4ef2-4a30-b208-c451ecf749d1"
 					(reference "C2")
+					(unit 1)
+				)
+			)
+		)
+	)
+	(symbol
+		(lib_id "Device:R_US")
+		(at 171.45 99.06 0)
+		(unit 1)
+		(exclude_from_sim no)
+		(in_bom yes)
+		(on_board yes)
+		(dnp no)
+		(property "Reference" "R1"
+			(at 173.482 98.298 0)
+			(effects
+				(font
+					(size 1.27 1.27)
+				)
+				(justify left)
+			)
+		)
+		(property "Value" "10k"
+			(at 173.736 100.076 0)
+			(effects
+				(font
+					(size 1 1)
+				)
+				(justify left)
+			)
+		)
+		(property "Footprint" "Resistor_THT:R_Axial_DIN0207_L6.3mm_D2.5mm_P7.62mm_Horizontal"
+			(at 172.466 99.314 90)
+			(effects
+				(font
+					(size 1.27 1.27)
+				)
+				(hide yes)
+			)
+		)
+		(property "Datasheet" "~"
+			(at 171.45 99.06 0)
+			(effects
+				(font
+					(size 1.27 1.27)
+				)
+				(hide yes)
+			)
+		)
+		(property "Description" ""
+			(at 171.45 99.06 0)
+			(effects
+				(font
+					(size 1.27 1.27)
+				)
+				(hide yes)
+			)
+		)
+		(pin "1"
+		)
+		(pin "2"
+		)
+		(instances
+			(project "pwm_driver_kicad"
+				(path "/d8411f75-4ef2-4a30-b208-c451ecf749d1"
+					(reference "R1")
 					(unit 1)
 				)
@@
 	(symbol
 		(lib_id "Simulation_SPICE:NMOS")
-		(at 175.26 95.25 0)
+		(at 179.07 95.25 0)
 		(unit 1)
 		(exclude_from_sim no)
@@
 		(dnp no)
 		(property "Reference" "Q1"
-			(at 179.07 90.17 0)
+			(at 182.88 90.17 0)
 			(effects
 				(font
@@
 		)
 		(property "Value" "IRF1407"
-			(at 179.07 92.202 0)
+			(at 182.88 92.202 0)
 			(effects
 				(font
@@
 		)
 		(property "Footprint" "Package_TO_SOT_THT:TO-220-3_Vertical"
-			(at 180.34 92.71 0)
+			(at 184.15 92.71 0)
 			(effects
 				(font
@@
 		)
 		(property "Datasheet" "https://ngspice.sourceforge.io/docs/ngspice-manual.pdf"
-			(at 175.26 107.95 0)
+			(at 179.07 107.95 0)
 			(effects
 				(font
@@
 		)
 		(property "Description" ""
-			(at 175.26 95.25 0)
+			(at 179.07 95.25 0)
 			(effects
 				(font
@@
 		)
 		(property "Sim.Device" "SUBCKT"
-			(at 175.26 112.395 0)
+			(at 179.07 112.395 0)
 			(effects
 				(font
@@
 		)
 		(property "Sim.Pins" "1=1 2=2 3=3"
-			(at 175.26 110.49 0)
+			(at 179.07 110.49 0)
 			(effects
 				(font
@@
 		)
 		(property "Sim.Library" "${KIPRJMOD}/pwm_driver_spice_simulation_models/IRF1407.spi"
-			(at 175.26 95.25 0)
+			(at 179.07 95.25 0)
 			(effects
 				(font
@@
 		)
 		(property "Sim.Name" "irf1407"
-			(at 175.26 95.25 0)
+			(at 179.07 95.25 0)
 			(effects
 				(font
@@
 			)
 		)
-		(property "Value" "0"
+		(property "Value" "GND"
 			(at 98.552 107.442 0)
 			(effects

Commit message: fix mosfet footprint pinout
Parts:
- added D3: LED, symbol Device:LED
- added R3: 220, Resistor_THT:R_Axial_DIN0207_L6.3mm_D2.5mm_P7.62mm_Horizontal, symbol Device:R_US
- Q1: value IRF1407 -> IRF540
Connections:
- net VCC: now also D3.1 (K)
- net at J1.1 (Pin_3), Q1.1 (D): now also R3.2
- new net: D3.2 (A), R3.1

Commit message: add led spice model: `pwm_driver_spice_simulation_models/led.lib`
Parts:
- R3: value 220 -> 330
Changed lines of the file:
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@@
+			)
+		)
+		(property "Sim.Library" "pwm_driver_spice_simulation_models/led.lib"
+			(at 189.23 72.39 0)
+			(effects
+				(font
+					(size 1.27 1.27)
+				)
+				(hide yes)
+			)
+		)
+		(property "Sim.Name" "LED2"
+			(at 189.23 72.39 0)
+			(effects
+				(font
+					(size 1.27 1.27)
+				)
+				(hide yes)
 			)
 		)
@@
 			)
 		)
-		(property "Sim.Params" "r=50k pos=0.75"
+		(property "Sim.Params" "r=50k pos=0.5"
 			(at 160.02 105.41 0)
 			(effects
@@
 			)
 		)
-		(property "Value" "220"
+		(property "Value" "330"
 			(at 191.516 82.296 0)
 			(effects

Commit message: replace third party 3D potentiometer model with own design
Other:
- moved on the sheet: B1, D3, J1, R3

Commit message: add simulation csv files
Other:
- note added: ".tran 10u 1m"
- note removed: ".tran 10u 2m"
Changed lines of the file:
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@@
 		)
 	)
-	(text ".tran 10u 2m"
+	(text ".tran 10u 1m"
 		(exclude_from_sim no)
 		(at 149.86 124.46 0)
